File: Binary_Counter.kicad_pcb (KiCad board)
At the start: 2 copper layers, 95.5 x 15 mm, 40 parts, among them J2 Conn_01x03_Pin, SW2 SW_MEC_5E, U1 CH32V003FxUx, U2 XC6206PxxxMR

Commit message: add LED holes
Parts:
- added ?: , TurboCase:CaseCorner_M3, F.Cu at (248.0, 105.5)
- added ?: , TurboCase:CaseCorner_M3, F.Cu at (123.0, 105.5)
- added ?: , TurboCase:CaseCorner_M3, F.Cu at (248.0, 80.5)
- added ?: , TurboCase:CaseCorner_M3, F.Cu at (123.0, 80.5)
